File: version_0.1/uSeqAnalogOuts.kicad_sch (KiCad schematic)
At the start: 130 parts, among them J1 Out A1, J11 Conn_01x04, J2 Out A2, J3 Out A3, J4 Out A4, J5 Out A5, J6 Out A7, J7 Out A6, J8 Out A8, J9 Conn_01x20, U1 TL072, U2 CJ431 SOT-23, U3 CJ431 SOT-23, U4 TL072, U5 CJ431 SOT-23, U6 CJ431 SOT-23, U7 TL072, U8 TL072

Commit message: 2024-07-03 save point
two output channels test layout.
Parts:
- D1: value LED A3 -> LED A4
- D2: value LED A1 -> LED A5
- D5: value LED A2 -> LED A6
- D6: value LED A3 -> LED A7
- D8: value LED A3 -> LED A8
- H1: footprint Connector_PinHeader_2.54mm:PinHeader_2x05_P2.54mm_Vertical_SMD -> Connector_PinHeader_2.54mm:PinHeader_2x05_P2.54mm_Vertical
Changed lines of the file:
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@@
 		(fields_autoplaced yes)
 		(property "Reference" "D2"
-			(at 49.8475 61.0067 0)
+			(at 49.8475 59.69 0)
 			(effects
 				(font
@@
 			)
 		)
-		(property "Value" "LED A1"
-			(at 49.8475 63.4309 0)
+		(property "Value" "LED A5"
+			(at 49.8475 62.23 0)
 			(effects
 				(font
@@
 		(fields_autoplaced yes)
 		(property "Reference" "D8"
-			(at 49.8475 90.2167 0)
+			(at 49.8475 88.9 0)
 			(effects
 				(font
@@
 			)
 		)
-		(property "Value" "LED A3"
-			(at 49.8475 92.6409 0)
+		(property "Value" "LED A8"
+			(at 49.8475 91.44 0)
 			(effects
 				(font
@@
 			)
 		)
-		(property "Footprint" "Connector_PinHeader_2.54mm:PinHeader_2x05_P2.54mm_Vertical_SMD"
+		(property "Footprint" "Connector_PinHeader_2.54mm:PinHeader_2x05_P2.54mm_Vertical"
 			(at 67.31 373.634 0)
 			(effects
@@
 		(fields_autoplaced yes)
 		(property "Reference" "D1"
-			(at 49.8475 50.8467 0)
+			(at 49.8475 49.53 0)
 			(effects
 				(font
@@
 			)
 		)
-		(property "Value" "LED A3"
-			(at 49.8475 53.2709 0)
+		(property "Value" "LED A4"
+			(at 49.8475 52.07 0)
 			(effects
 				(font
@@
 		(fields_autoplaced yes)
 		(property "Reference" "D5"
-			(at 49.8475 70.1507 0)
+			(at 49.8475 69.85 0)
 			(effects
 				(font
@@
 			)
 		)
-		(property "Value" "LED A2"
-			(at 49.8475 72.5749 0)
+		(property "Value" "LED A6"
+			(at 49.8475 72.39 0)
 			(effects
 				(font
@@
 		(fields_autoplaced yes)
 		(property "Reference" "D6"
-			(at 49.8475 80.0567 0)
+			(at 49.8475 78.74 0)
 			(effects
 				(font
@@
 			)
 		)
-		(property "Value" "LED A3"
-			(at 49.8475 82.4809 0)
+		(property "Value" "LED A7"
+			(at 49.8475 81.28 0)
 			(effects
 				(font
